File: XBox button board/XBox button board.kicad_pcb (KiCad board)
At the start: 2 copper layers, 80 x 40.6 mm, 16 parts, among them J1 Conn_01x09_Pin, J2 Conn_01x03

Commit message: Minor image adjustment
moved some graphics
Parts:
- moved G*** 11.9 mm to (118.5, 110.1)
Changed lines of the file:
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@@
 	(footprint "LOGO"
 		(layer "F.Cu")
-		(at 129.55 114.5)
+		(at 118.45 110.1)
 		(property "Reference" "G***"
 			(at 0 0 0)

Commit message: updated silkscreens
removed logos from silk print area
Parts:
- moved G*** 11.5 mm to (175.3, 112.0)
- moved G*** 4.72 mm to (116.9, 105.6)
- moved G*** 2.32 mm to (116.1, 115.1)
- moved G*** 1.83 mm to (116.7, 110.5)
Changed lines of the file:
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@@
 	(footprint "LOGO"
 		(layer "F.Cu")
-		(at 118.390611 114.828508)
+		(at 116.090611 115.128508)
 		(property "Reference" "G***"
 			(at 0 0 0)
@@
 	(footprint "LOGO"
 		(layer "F.Cu")
-		(at 170.254788 101.693806)
+		(at 175.35 112)
 		(property "Reference" "G***"
 			(at 0 0 0)
@@
 	(footprint "LOGO"
 		(layer "F.Cu")
-		(at 118.45 110.1)
+		(at 116.65 110.45)
 		(property "Reference" "G***"
 			(at 0 0 0)
@@
 	(footprint "LOGO"
 		(layer "F.Cu")
-		(at 118.61083 101.2)
+		(at 116.9 105.6)
 		(property "Reference" "G***"
 			(at 0 0 0)
