File: XBox button board - no HDD-LAN/XBox button board_no_LAN-HDD.kicad_pcb (KiCad board)
At the start: 2 copper layers, 80 x 40.6 mm, 9 parts, among them J1 Conn_01x09_Pin

Commit message: Minor image adjustment
moved some graphics
Parts:
- moved G*** 12.1 mm to (118.3, 110.1)
Changed lines of the file:
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@@
 	(footprint "LOGO"
 		(layer "F.Cu")
-		(at 129.55 114.5)
+		(at 118.3 110.1)
 		(property "Reference" "G***"
 			(at 0 0 0)

Commit message: updated silkscreens
removed logos from silk print area
Parts:
- moved G*** 4.56 mm to (117.0, 105.5)
- moved G*** 4.52 mm to (172.2, 105.8)
Changed lines of the file:
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@@
 	(footprint "LOGO"
 		(layer "F.Cu")
-		(at 170.254788 101.693806)
+		(at 172.25 105.75)
 		(property "Reference" "G***"
 			(at 0 0 0)
@@
 	(footprint "LOGO"
 		(layer "F.Cu")
-		(at 118.61083 101.2)
+		(at 116.95 105.45)
 		(property "Reference" "G***"
 			(at 0 0 0)
